Commit message: chore: repository cleanup

File: src/Tyre_Inspection_Bot/src/amr_hardware/src/ugv_description/urdf/ugv_rover.urdf (robot description, URDF)
Before this commit: robot ugv_rover, 17 links, 16 joints
Links:
- removed link base_footprint
- removed link camera_depth_optical_frame
Joints:
- removed joint base_joint
- removed joint camera_depth_optical_joint
